File: P26_ESP32_Motors.sch (KiCad schematic (older format))
At the start: 5 parts

Commit message: Added components.
Smaller changes.
Parts:
- added D? (x3): D_Zener, symbol Device:D_Zener
- added J? (x3): Screw_Terminal_01x02, symbol Connector:Screw_Terminal_01x02
- added Q? (x3): Q_NMOS_DGS, symbol Device:Q_NMOS_DGS
- added R? (x3): R, symbol Device:R
- added R? (x3): 1K, symbol Device:R
Connections:
- wire segments 13 -> 52

Commit message: Naming components and adding global labels
Parts:
- D203: renamed from D?; footprint (none) -> Package_SO:SOIC-8_3.9x4.9mm_P1.27mm
- R201: renamed from R10; value 1K -> 270
- R202, R203, R204: renamed from R?; value 1K -> 270
- R204, R207, R208: renamed from R?; value R -> 10K
- R?: value R -> 10K
- gave numbers to parts that had none: 11
Connections:
- net labels added: MOTOR1, MOTOR2, MOTOR3, MOTOR4
Changed lines of the file:
@@
 $EndDescr
 $Comp
-L Device:Q_NMOS_DGS Q?
+L Device:Q_NMOS_DGS Q201
 U 1 1 5B07320A
 P 4350 2350
-F 0 "Q?" H 4555 2396 50  0000 L CNN
+F 0 "Q201" H 4555 2396 50  0000 L CNN
 F 1 "Q_NMOS_DGS" H 4555 2305 50  0000 L CNN
 F 2 "" H 4550 2450 50  0001 C CNN
@@
 $EndComp
 $Comp
-L Device:R R?
+L Device:R R204
 U 1 1 5B073576
 P 4000 2650
-F 0 "R?" H 4070 2696 50  0000 L CNN
-F 1 "R" H 4070 2605 50  0000 L CNN
+F 0 "R204" H 4070 2696 50  0000 L CNN
+F 1 "10K" H 4070 2605 50  0000 L CNN
 F 2 "" V 3930 2650 50  0001 C CNN
 F 3 "~" H 4000 2650 50  0001 C CNN
@@
 $EndComp
 $Comp
-L Device:R R10
+L Device:R R201
 U 1 1 5B07369A
 P 3500 2350
-F 0 "R10" H 3570 2396 50  0000 L CNN
-F 1 "1K" H 3570 2305 50  0000 L CNN
+F 0 "R201" H 3570 2396 50  0000 L CNN
+F 1 "270" H 3570 2305 50  0000 L CNN
 F 2 "" V 3430 2350 50  0001 C CNN
 F 3 "~" H 3500 2350 50  0001 C CNN
@@
 $EndComp
 $Comp
-L Device:D_Zener D?
+L Device:D_Zener D201
 U 1 1 5B07375C
 P 3750 2650
-F 0 "D?" V 3704 2729 50  0000 L CNN
+F 0 "D201" V 3704 2729 50  0000 L CNN
 F 1 "D_Zener" V 3795 2729 50  0000 L CNN
 F 2 "" H 3750 2650 50  0001 C CNN
@@
 	4000 2950 4000 3000
 $Comp
-L Connector:Screw_Terminal_01x02 J?
+L Connector:Screw_Terminal_01x02 J201
 U 1 1 5B06C162
 P 4650 1950
-F 0 "J?" H 4730 1942 50  0000 L CNN
+F 0 "J201" H 4730 1942 50  0000 L CNN
 F 1 "Screw_Terminal_01x02" H 4730 1851 50  0000 L CNN
 F 2 "" H 4650 1950 50  0001 C CNN
@@
 	4450 1400 4450 1950
 $Comp
-L Device:Q_NMOS_DGS Q?
+L Device:Q_NMOS_DGS Q203
 U 1 1 5B361E3C
 P 7500 2350
-F 0 "Q?" H 7705 2396 50  0000 L CNN
+F 0 "Q203" H 7705 2396 50  0000 L CNN
 F 1 "Q_NMOS_DGS" H 7705 2305 50  0000 L CNN
 F 2 "" H 7700 2450 50  0001 C CNN
@@
 $EndComp
 $Comp
-L Device:R R?
+L Device:R R207
 U 1 1 5B361E43
 P 7150 2650
-F 0 "R?" H 7220 2696 50  0000 L CNN
-F 1 "R" H 7220 2605 50  0000 L CNN
+F 0 "R207" H 7220 2696 50  0000 L CNN
+F 1 "10K" H 7220 2605 50  0000 L CNN
 F 2 "" V 7080 2650 50  0001 C CNN
 F 3 "~" H 7150 2650 50  0001 C CNN
@@
 $EndComp
 $Comp
-L Device:R R?
+L Device:R R203
 U 1 1 5B361E4A
 P 6650 2350
-F 0 "R?" H 6720 2396 50  0000 L CNN
-F 1 "1K" H 6720 2305 50  0000 L CNN
+F 0 "R203" H 6720 2396 50  0000 L CNN
+F 1 "270" H 6720 2305 50  0000 L CNN
 F 2 "" V 6580 2350 50  0001 C CNN
 F 3 "~" H 6650 2350 50  0001 C CNN
@@
 $EndComp
 $Comp
-L Device:D_Zener D?
+L Device:D_Zener D203
 U 1 1 5B361E51
 P 6900 2650
-F 0 "D?" V 6854 2729 50  0000 L CNN
+F 0 "D203" V 6854 2729 50  0000 L CNN
 F 1 "D_Zener" V 6945 2729 50  0000 L CNN
-F 2 "" H 6900 2650 50  0001 C CNN
+F 2 "Package_SO:SOIC-8_3.9x4.9mm_P1.27mm" H 6900 2650 50  0001 C CNN
 F 3 "~" H 6900 2650 50  0001 C CNN
 	1    6900 2650
@@
 	6800 2350 6900 2350
 Wire Wire Line
-	6500 2350 6300 2350
-Wire Wire Line
 	7150 2800 7150 2950
 Wire Wire Line
@@
 	7150 2950 7150 3000
 $Comp
-L Connector:Screw_Terminal_01x02 J?
+L Connector:Screw_Terminal_01x02 J203
 U 1 1 5B361E6D
 P 7800 1950
-F 0 "J?" H 7880 1942 50  0000 L CNN
+F 0 "J203" H 7880 1942 50  0000 L CNN
 F 1 "Screw_Terminal_01x02" H 7880 1851 50  0000 L CNN
 F 2 "" H 7800 1950 50  0001 C CNN
@@
 	7600 1400 7600 1950
 $Comp
-L Device:Q_NMOS_DGS Q?
+L Device:Q_NMOS_DGS Q202
 U 1 1 5B36240D
 P 4350 4750
-F 0 "Q?" H 4555 4796 50  0000 L CNN
+F 0 "Q202" H 4555 4796 50  0000 L CNN
 F 1 "Q_NMOS_DGS" H 4555 4705 50  0000 L CNN
 F 2 "" H 4550 4850 50  0001 C CNN
@@
 P 4000 5050
 F 0 "R?" H 4070 5096 50  0000 L CNN
-F 1 "R" H 4070 5005 50  0000 L CNN
+F 1 "10K" H 4070 5005 50  0000 L CNN
 F 2 "" V 3930 5050 50  0001 C CNN
 F 3 "~" H 4000 5050 50  0001 C CNN
@@
 $EndComp
 $Comp
-L Device:R R?
+L Device:R R202
 U 1 1 5B36241B
 P 3500 4750
-F 0 "R?" H 3570 4796 50  0000 L CNN
-F 1 "1K" H 3570 4705 50  0000 L CNN
+F 0 "R202" H 3570 4796 50  0000 L CNN
+F 1 "270" H 3570 4705 50  0000 L CNN
 F 2 "" V 3430 4750 50  0001 C CNN
 F 3 "~" H 3500 4750 50  0001 C CNN
@@
 $EndComp
 $Comp
-L Device:D_Zener D?
+L Device:D_Zener D202
 U 1 1 5B362422
 P 3750 5050
-F 0 "D?" V 3704 5129 50  0000 L CNN
+F 0 "D202" V 3704 5129 50  0000 L CNN
 F 1 "D_Zener" V 3795 5129 50  0000 L CNN
 F 2 "" H 3750 5050 50  0001 C CNN
@@
 	3650 4750 3750 4750
 Wire Wire Line
-	3350 4750 3150 4750
-Wire Wire Line
 	4000 5200 4000 5350
 Wire Wire Line
@@
 	4000 5350 4000 5400
 $Comp
-L Connector:Screw_Terminal_01x02 J?
+L Connector:Screw_Terminal_01x02 J202
 U 1 1 5B36243E
 P 4650 4350
-F 0 "J?" H 4730 4342 50  0000 L CNN
+F 0 "J202" H 4730 4342 50  0000 L CNN
 F 1 "Screw_Terminal_01x02" H 4730 4251 50  0000 L CNN
 F 2 "" H 4650 4350 50  0001 C CNN
@@
 	4450 3800 4450 4350
 $Comp
-L Device:Q_NMOS_DGS Q?
+L Device:Q_NMOS_DGS Q204
 U 1 1 5B36244D
 P 7500 4750
-F 0 "Q?" H 7705 4796 50  0000 L CNN
+F 0 "Q204" H 7705 4796 50  0000 L CNN
 F 1 "Q_NMOS_DGS" H 7705 4705 50  0000 L CNN
 F 2 "" H 7700 4850 50  0001 C CNN
@@
 $EndComp
 $Comp
-L Device:R R?
+L Device:R R208
 U 1 1 5B362454
 P 7150 5050
-F 0 "R?" H 7220 5096 50  0000 L CNN
-F 1 "R" H 7220 5005 50  0000 L CNN
+F 0 "R208" H 7220 5096 50  0000 L CNN
+F 1 "10K" H 7220 5005 50  0000 L CNN
 F 2 "" V 7080 5050 50  0001 C CNN
 F 3 "~" H 7150 5050 50  0001 C CNN
@@
 $EndComp
 $Comp
-L Device:R R?
+L Device:R R204
 U 1 1 5B36245B
 P 6650 4750
-F 0 "R?" H 6720 4796 50  0000 L CNN
-F 1 "1K" H 6720 4705 50  0000 L CNN
+F 0 "R204" H 6720 4796 50  0000 L CNN
+F 1 "270" H 6720 4705 50  0000 L CNN
 F 2 "" V 6580 4750 50  0001 C CNN
 F 3 "~" H 6650 4750 50  0001 C CNN
@@
 $EndComp
 $Comp
-L Device:D_Zener D?
+L Device:D_Zener D204
 U 1 1 5B362462
 P 6900 5050
-F 0 "D?" V 6854 5129 50  0000 L CNN
+F 0 "D204" V 6854 5129 50  0000 L CNN
 F 1 "D_Zener" V 6945 5129 50  0000 L CNN
 F 2 "" H 6900 5050 50  0001 C CNN
@@
 	6800 4750 6900 4750
 Wire Wire Line
-	6500 4750 6300 4750
-Wire Wire Line
 	7150 5200 7150 5350
 Wire Wire Line
@@
 	7150 5350 7150 5400
 $Comp
-L Connector:Screw_Terminal_01x02 J?
+L Connector:Screw_Terminal_01x02 J204
 U 1 1 5B36247E
 P 7800 4350
-F 0 "J?" H 7880 4342 50  0000 L CNN
+F 0 "J204" H 7880 4342 50  0000 L CNN
 F 1 "Screw_Terminal_01x02" H 7880 4251 50  0000 L CNN
 F 2 "" H 7800 4350 50  0001 C CNN
@@
 Wire Wire Line
 	7600 3800 7600 4350
+Text GLabel 3150 2350 0    50   Input ~ 0
+MOTOR1
+Text GLabel 3150 4750 0    50   Input ~ 0
+MOTOR2
+Text GLabel 6150 2350 0    50   Input ~ 0
+MOTOR3
+Wire Wire Line
+	6150 2350 6500 2350
+Text GLabel 6100 4750 0    50   Input ~ 0
+MOTOR4
+Wire Wire Line
+	6100 4750 6500 4750
+Wire Wire Line
+	3350 4750 3150 4750
 $EndSCHEMATC
